File: hardware/electronic/MK1/power.sch (KiCad schematic (older format))
At the start: 3 parts

Commit message: HW: First placement of MCU and headers
Parts:
- gave numbers to parts that had none: 3
Changed lines of the file:
@@
 $EndDescr
 $Comp
-L Battery BT?
+L Battery BT1
 U 1 1 5885FA38
 P 1900 1550
-F 0 "BT?" H 2000 1600 50  0000 L CNN
+F 0 "BT1" H 2000 1600 50  0000 L CNN
 F 1 "Battery" H 2000 1500 50  0000 L CNN
-F 2 "" V 1900 1590 50  0000 C CNN
+F 2 "" V 1900 1590 50  0001 C CNN
 F 3 "" V 1900 1590 50  0000 C CNN
 	1    1900 1550
@@
 $EndComp
 $Comp
-L GND #PWR?
+L GND #PWR06
 U 1 1 5885FB0A
 P 1900 1700
-F 0 "#PWR?" H 1900 1450 50  0001 C CNN
+F 0 "#PWR06" H 1900 1450 50  0001 C CNN
 F 1 "GND" H 1900 1550 50  0000 C CNN
 F 2 "" H 1900 1700 50  0000 C CNN
@@
 VBAT
 $Comp
-L R R?
+L R R3
 U 1 1 5885FCA2
 P 4000 1550
-F 0 "R?" V 4080 1550 50  0000 C CNN
+F 0 "R3" V 4080 1550 50  0000 C CNN
 F 1 "5k" V 4000 1550 50  0000 C CNN
-F 2 "" V 3930 1550 50  0000 C CNN
+F 2 "" V 3930 1550 50  0001 C CNN
 F 3 "" H 4000 1550 50  0000 C CNN
 	1    4000 1550
@@
 $EndComp
 $Comp
-L R R?
+L R R4
 U 1 1 5885FCD9
 P 4000 1950
-F 0 "R?" V 4080 1950 50  0000 C CNN
+F 0 "R4" V 4080 1950 50  0000 C CNN
 F 1 "10k" V 4000 1950 50  0000 C CNN
-F 2 "" V 3930 1950 50  0000 C CNN
+F 2 "" V 3930 1950 50  0001 C CNN
 F 3 "" H 4000 1950 50  0000 C CNN
 	1    4000 1950
@@
 Connection ~ 4000 1750
 $Comp
-L GND #PWR?
+L GND #PWR07
 U 1 1 5885FD97
 P 4000 2100
-F 0 "#PWR?" H 4000 1850 50  0001 C CNN
+F 0 "#PWR07" H 4000 1850 50  0001 C CNN
 F 1 "GND" H 4000 1950 50  0000 C CNN
 F 2 "" H 4000 2100 50  0000 C CNN

Commit message: HW: Add VL53L0X carrier
Parts:
- R3, R4: footprint (none) -> Resistors_SMD:R_0805
Changed lines of the file:
@@
 $Descr A4 11693 8268
 encoding utf-8
-Sheet 4 5
+Sheet 4 6
 Title "O'PAVES Mk-I"
 Date ""
@@
 F 0 "R3" V 4080 1550 50  0000 C CNN
 F 1 "5k" V 4000 1550 50  0000 C CNN
-F 2 "" V 3930 1550 50  0001 C CNN
+F 2 "Resistors_SMD:R_0805" V 3930 1550 50  0001 C CNN
 F 3 "" H 4000 1550 50  0000 C CNN
 	1    4000 1550
@@
 F 0 "R4" V 4080 1950 50  0000 C CNN
 F 1 "10k" V 4000 1950 50  0000 C CNN
-F 2 "" V 3930 1950 50  0001 C CNN
+F 2 "Resistors_SMD:R_0805" V 3930 1950 50  0001 C CNN
 F 3 "" H 4000 1950 50  0000 C CNN
 	1    4000 1950
