File: hardware/electronic/MK1/imu.sch (KiCad schematic (older format))
At the start: 9 parts, among them U3 Bosch_BNO055_IMU, U4 AdaFruit_BNO055_Breakout, Y2 Crystal

Commit message: HW: Minor cleanup in the schematics and layout
Other:
- note added: "IMU"
Changed lines of the file:
@@
 encoding utf-8
 Sheet 7 7
-Title ""
+Title "O'PAVES Mk-I"
 Date ""
-Rev ""
-Comp ""
+Rev "A"
+Comp "AdaCore"
 Comment1 ""
 Comment2 ""
@@
 Text Notes 7550 1550 0    59   ~ 0
 If for some reason it's not possible to use the on-board \nIMU (bad circuit, too difficult to solder, etc) we will use \na breakout board from AdaFruit.
+Text Notes 3100 1400 0    394  ~ 0
+IMU
 $EndSCHEMATC

Commit message: HW: Add missing component values
Parts:
- Y2: value Crystal -> 32kHz
Changed lines of the file:
@@
 P 1700 5250
 F 0 "Y2" H 1700 5400 50  0000 C CNN
-F 1 "Crystal" H 1700 5100 50  0000 C CNN
+F 1 "32kHz" H 1700 5100 50  0000 C CNN
 F 2 "Crystals:Crystal_HC50-U_Vertical" H 1700 5250 50  0001 C CNN
 F 3 "" H 1700 5250 50  0000 C CNN

Commit message: HW: Change crystal footprints
Parts:
- Y2: footprint Crystals:Crystal_HC50-U_Vertical -> Crystals:Crystal_MC-306
Changed lines of the file:
@@
 F 0 "Y2" H 1700 5400 50  0000 C CNN
 F 1 "32kHz" H 1700 5100 50  0000 C CNN
-F 2 "Crystals:Crystal_HC50-U_Vertical" H 1700 5250 50  0001 C CNN
+F 2 "Crystals:Crystal_MC-306" H 1700 5250 50  0001 C CNN
 F 3 "" H 1700 5250 50  0000 C CNN
 	1    1700 5250
