File: hardware/electronic/MK1/imu.sch (KiCad schematic (older format))
At the start: 9 parts, among them U3 Bosch_BNO055_IMU, U4 AdaFruit_BNO055_Breakout, Y2 32kHz

Commit message: HW: Connect the NRESET pin of the IMU to the MCU
Parts:
- removed R6: 10k, Resistors_SMD:R_0805, symbol R
Connections:
- net IMU_NRST: now reaches U3.11 (nRESET)
- net IMU_NRST: now also U4.6 (RST)
- no-connect marks 17 -> 16
Changed lines of the file:
@@
 $EndComp
 $Comp
-L GND #PWR34
+L GND #PWR029
 U 1 1 5886F001
 P 3200 5650
-F 0 "#PWR34" H 3200 5400 50  0001 C CNN
+F 0 "#PWR029" H 3200 5400 50  0001 C CNN
 F 1 "GND" H 3200 5500 50  0000 C CNN
 F 2 "" H 3200 5650 50  0000 C CNN
@@
 Connection ~ 3850 5450
 $Comp
-L GND #PWR35
+L GND #PWR030
 U 1 1 5886F07C
 P 3850 5600
-F 0 "#PWR35" H 3850 5350 50  0001 C CNN
+F 0 "#PWR030" H 3850 5350 50  0001 C CNN
 F 1 "GND" H 3850 5450 50  0000 C CNN
 F 2 "" H 3850 5600 50  0000 C CNN
@@
 Connection ~ 1850 3800
 $Comp
-L GND #PWR31
+L GND #PWR031
 U 1 1 5886F184
 P 1850 3850
-F 0 "#PWR31" H 1850 3600 50  0001 C CNN
+F 0 "#PWR031" H 1850 3600 50  0001 C CNN
 F 1 "GND" H 1850 3700 50  0000 C CNN
 F 2 "" H 1850 3850 50  0000 C CNN
@@
 $EndComp
 $Comp
-L GND #PWR36
+L GND #PWR032
 U 1 1 5886F3DB
 P 4200 2300
-F 0 "#PWR36" H 4200 2050 50  0001 C CNN
+F 0 "#PWR032" H 4200 2050 50  0001 C CNN
 F 1 "GND" H 4200 2150 50  0000 C CNN
 F 2 "" H 4200 2300 50  0000 C CNN
@@
 Connection ~ 1700 5800
 $Comp
-L GND #PWR30
+L GND #PWR033
 U 1 1 5886F8B7
 P 1700 5900
-F 0 "#PWR30" H 1700 5650 50  0001 C CNN
+F 0 "#PWR033" H 1700 5650 50  0001 C CNN
 F 1 "GND" H 1700 5750 50  0000 C CNN
 F 2 "" H 1700 5900 50  0000 C CNN
@@
 $EndComp
 $Comp
-L GND #PWR33
+L GND #PWR034
 U 1 1 5886FCA1
 P 2100 4300
-F 0 "#PWR33" H 2100 4050 50  0001 C CNN
+F 0 "#PWR034" H 2100 4050 50  0001 C CNN
 F 1 "GND" H 2100 4150 50  0000 C CNN
 F 2 "" H 2100 4300 50  0000 C CNN
@@
 	0    1    1    0
 $EndComp
-$Comp
-L R R6
-U 1 1 5886FDF0
-P 1650 2600
-F 0 "R6" V 1730 2600 50  0000 C CNN
-F 1 "10k" V 1650 2600 50  0000 C CNN
-F 2 "Resistors_SMD:R_0805" V 1580 2600 50  0001 C CNN
-F 3 "" H 1650 2600 50  0000 C CNN
-	1    1650 2600
-	1    0    0    -1
-$EndComp
-Wire Wire Line
-	2100 2950 1650 2950
-Wire Wire Line
-	1650 2950 1650 2750
 Text HLabel 3450 2300 1    60   Input ~ 0
 IMU_VCC
-Text HLabel 1650 2300 1    60   Input ~ 0
+Text HLabel 1350 2350 1    60   Input ~ 0
 IMU_VCC
-Wire Wire Line
-	1650 2450 1650 2300
 $Comp
 L R R5
@@
 	1350 2450 1350 2350
 Wire Wire Line
-	1350 2350 1650 2350
-Connection ~ 1650 2350
-Wire Wire Line
 	2100 3150 1350 3150
 Wire Wire Line
 	1350 3150 1350 2750
 $Comp
-L GND #PWR32
+L GND #PWR035
 U 1 1 58870499
 P 2100 4150
-F 0 "#PWR32" H 2100 3900 50  0001 C CNN
+F 0 "#PWR035" H 2100 3900 50  0001 C CNN
 F 1 "GND" H 2100 4000 50  0000 C CNN
 F 2 "" H 2100 4150 50  0000 C CNN
@@
 Text HLabel 7050 3050 0    60   BiDi ~ 0
 IMU_SDA
-NoConn ~ 7050 2800
 NoConn ~ 7050 3450
 $Comp
-L GND #PWR37
+L GND #PWR036
 U 1 1 588A8ACC
 P 9050 4500
-F 0 "#PWR37" H 9050 4250 50  0001 C CNN
+F 0 "#PWR036" H 9050 4250 50  0001 C CNN
 F 1 "GND" H 9050 4350 50  0000 C CNN
 F 2 "" H 9050 4500 50  0000 C CNN
@@
 Text Notes 3100 1400 0    394  ~ 0
 IMU
+Text HLabel 1700 2350 1    60   Input ~ 0
+IMU_NRST
+Wire Wire Line
+	2100 2950 1700 2950
+Wire Wire Line
+	1700 2950 1700 2350
+Text HLabel 7050 2800 0    60   Input ~ 0
+IMU_NRST
 $EndSCHEMATC

Commit message: HW: Fix BNO055 pin 10 to GND
Connections:
- net GND: now also U3.2 (GND)
- net at U3.9 (CAP): now also C15.1
- no-connect marks 16 -> 15
Other:
- moved on the sheet: C15
Changed lines of the file:
@@
 L C_Small C15
 U 1 1 5886EF60
-P 3200 5550
-F 0 "C15" H 3210 5620 50  0000 L CNN
-F 1 "100nF" H 3210 5470 50  0000 L CNN
-F 2 "Capacitors_SMD:C_0805" H 3200 5550 50  0001 C CNN
-F 3 "" H 3200 5550 50  0000 C CNN
-	1    3200 5550
+P 2950 5550
+F 0 "C15" H 2960 5620 50  0000 L CNN
+F 1 "100nF" H 2960 5470 50  0000 L CNN
+F 2 "Capacitors_SMD:C_0805" H 2950 5550 50  0001 C CNN
+F 3 "" H 2950 5550 50  0000 C CNN
+	1    2950 5550
 	1    0    0    -1
 $EndComp
@@
 L GND #PWR029
 U 1 1 5886F001
-P 3200 5650
-F 0 "#PWR029" H 3200 5400 50  0001 C CNN
-F 1 "GND" H 3200 5500 50  0000 C CNN
-F 2 "" H 3200 5650 50  0000 C CNN
-F 3 "" H 3200 5650 50  0000 C CNN
-	1    3200 5650
-	1    0    0    -1
-$EndComp
-Wire Wire Line
-	3550 5450 4150 5450
+P 2950 5650
+F 0 "#PWR029" H 2950 5400 50  0001 C CNN
+F 1 "GND" H 2950 5500 50  0000 C CNN
+F 2 "" H 2950 5650 50  0000 C CNN
+F 3 "" H 2950 5650 50  0000 C CNN
+	1    2950 5650
+	1    0    0    -1
+$EndComp
+Wire Wire Line
+	3350 5450 4150 5450
 Connection ~ 3750 5450
 Connection ~ 3950 5450
@@
 $EndComp
 NoConn ~ 2100 2750
-NoConn ~ 2100 3350
 NoConn ~ 5100 3350
 NoConn ~ 5100 3500
@@
 Text HLabel 7050 2800 0    60   Input ~ 0
 IMU_NRST
+Connection ~ 3550 5450
 $EndSCHEMATC
