File: hardware/electronic/MK2/microcontroller.sch (KiCad schematic (older format))
At the start: 6 parts, among them P1 CF_EXP_LEFT, P2 CF_EXP_RIGHT, P3 CONN_01X04, U2 MCP23008

Commit message: HW: Update Mk-II design
Parts:
- removed R11, R12: 10k, Resistors_SMD:R_0805, symbol R
- added C1: C, Capacitors_ThroughHole:C_Disc_D7.5_P5, symbol C
- added JP1: Jumper_NO_Small, Resistors_SMD:R_0805_HandSoldering, symbol Jumper_NO_Small
- renumbered P3 to P2, P2 to P3, U2 to U3
Connections:
- net 5V: now also P3.10 (VUSB)
- net GND: now also C1.2
- net MCU_VCC: now also C1.1, JP1.2; no longer P3.10 (VUSB)
- net at P1.1 (VCC): now also JP1.1
- net Encoder_A: no longer names the net of P1.9 (IO_4)
- net Encoder_B: no longer names the net of P3.5 (MOSI)
Other:
- note removed: "Pull-UPs"
Changed lines of the file:
@@
 Title "O'PAVES Mk-II"
 Date ""
-Rev "A"
+Rev "B"
 Comp "AdaCore"
 Comment1 "Licensed under CERN OHL v.1.2 or later"
@@
 $EndDescr
 Text HLabel 8450 4750 2    60   Input ~ 0
-MCU_VCC
+5V
 Text HLabel 8450 4150 2    60   Input ~ 0
 VBAT_SENSE
-Wire Notes Line
-	550  8950 11800 8950
-Wire Notes Line
-	3650 8950 3650 11200
-Wire Notes Line
-	7950 8950 7950 11200
 Text HLabel 5950 4250 2    60   Input ~ 0
 Distance_SCL
 Text HLabel 5950 4150 2    60   Input ~ 0
 Distance_SDA
-Wire Notes Line
-	11800 8950 11800 9950
-Text Notes 10100 9250 0    118  ~ 0
-Pull-UPs
-$Comp
-L R R11
-U 1 1 5891BCC4
-P 10350 10300
-F 0 "R11" V 10430 10300 50  0000 C CNN
-F 1 "10k" V 10350 10300 50  0000 C CNN
-F 2 "Resistors_SMD:R_0805" V 10280 10300 50  0001 C CNN
-F 3 "" H 10350 10300 50  0000 C CNN
-	1    10350 10300
-	1    0    0    -1
-$EndComp
-$Comp
-L R R12
-U 1 1 5891BCCA
-P 10650 10300
-F 0 "R12" V 10730 10300 50  0000 C CNN
-F 1 "10k" V 10650 10300 50  0000 C CNN
-F 2 "Resistors_SMD:R_0805" V 10580 10300 50  0001 C CNN
-F 3 "" H 10650 10300 50  0000 C CNN
-	1    10650 10300
-	1    0    0    -1
-$EndComp
-Wire Wire Line
-	10350 10150 10650 10150
-Wire Wire Line
-	10500 10150 10500 9950
-Connection ~ 10500 10150
-Text HLabel 10500 9950 1    60   Input ~ 0
-MCU_VCC
-Text HLabel 10350 10450 3    60   Input ~ 0
-Distance_SCL
-Text HLabel 10650 10450 3    60   Input ~ 0
-Distance_SDA
-Text HLabel 5950 4650 2    60   Input ~ 0
-Encoder_A
-Text HLabel 8450 4250 2    60   Input ~ 0
-Encoder_B
 Text HLabel 8450 3850 2    60   Input ~ 0
 Motor_PWMA
@@
 $EndComp
 $Comp
-L CF_EXP_RIGHT P2
+L CF_EXP_RIGHT P3
 U 1 1 5984C362
 P 7750 4300
-F 0 "P2" H 7750 3750 60  0000 C CNN
+F 0 "P3" H 7750 3750 60  0000 C CNN
 F 1 "CF_EXP_RIGHT" H 7750 3650 60  0000 C CNN
 F 2 "crazyflie2-exp:CF2-DECK-SMD-HOLES" H 7900 3650 60  0001 C CNN
@@
 Distance_SDA
 $Comp
-L GND #PWR016
+L GND #PWR012
 U 1 1 5984DF0A
 P 8000 7050
-F 0 "#PWR016" H 8000 6800 50  0001 C CNN
+F 0 "#PWR012" H 8000 6800 50  0001 C CNN
 F 1 "GND" H 8000 6900 50  0000 C CNN
 F 2 "" H 8000 7050 50  0000 C CNN
@@
 $EndComp
 $Comp
-L GND #PWR017
+L GND #PWR013
 U 1 1 5984DF24
 P 5950 4750
-F 0 "#PWR017" H 5950 4500 50  0001 C CNN
+F 0 "#PWR013" H 5950 4500 50  0001 C CNN
 F 1 "GND" H 5950 4600 50  0000 C CNN
 F 2 "" H 5950 4750 50  0000 C CNN
@@
 Extern_TX
 $Comp
-L CONN_01X04 P3
+L CONN_01X04 P2
 U 1 1 5988473B
 P 5600 6300
-F 0 "P3" H 5600 6550 50  0000 C CNN
+F 0 "P2" H 5600 6550 50  0000 C CNN
 F 1 "CONN_01X04" V 5700 6300 50  0000 C CNN
 F 2 "Pin_Headers:Pin_Header_Straight_1x04" H 5600 6300 50  0001 C CNN
@@
 Extern_TX
 $Comp
-L GND #PWR018
+L GND #PWR014
 U 1 1 59884A46
 P 5400 6450
-F 0 "#PWR018" H 5400 6200 50  0001 C CNN
+F 0 "#PWR014" H 5400 6200 50  0001 C CNN
 F 1 "GND" H 5400 6300 50  0000 C CNN
 F 2 "" H 5400 6450 50  0000 C CNN
@@
 Motor_PWMB
 $Comp
-L MCP23008 U2
+L MCP23008 U3
 U 1 1 598C8911
 P 7400 5650
-F 0 "U2" H 7400 5650 60  0000 C CNN
+F 0 "U3" H 7400 5650 60  0000 C CNN
 F 1 "MCP23008" V 8100 4900 60  0000 C CNN
 F 2 "Housings_DIP:DIP-18_W7.62mm_LongPads" H 7400 5650 60  0001 C CNN
@@
 Connection ~ 7400 6350
 $Comp
-L GND #PWR019
+L GND #PWR015
 U 1 1 598C8AD6
 P 6700 6400
-F 0 "#PWR019" H 6700 6150 50  0001 C CNN
+F 0 "#PWR015" H 6700 6150 50  0001 C CNN
 F 1 "GND" H 6700 6250 50  0000 C CNN
 F 2 "" H 6700 6400 50  0000 C CNN
@@
 Text HLabel 8000 5750 1    60   Input ~ 0
 MCU_VCC
-Text HLabel 7400 6550 0    60   Input ~ 0
+Text HLabel 7050 6650 0    60   Input ~ 0
 MCU_VCC
 Wire Wire Line
 	6700 6350 6700 6400
+$Comp
+L C C1
+U 1 1 5A0F4B30
+P 7050 6800
+F 0 "C1" H 7075 6900 50  0000 L CNN
+F 1 "C" H 7075 6700 50  0000 L CNN
+F 2 "Capacitors_ThroughHole:C_Disc_D7.5_P5" H 7088 6650 50  0001 C CNN
+F 3 "" H 7050 6800 50  0000 C CNN
+	1    7050 6800
+	1    0    0    -1
+$EndComp
+Wire Wire Line
+	7050 6650 7050 6550
+Wire Wire Line
+	7050 6550 7400 6550
+$Comp
+L GND #PWR016
+U 1 1 5A0F4C63
+P 7050 7000
+F 0 "#PWR016" H 7050 6750 50  0001 C CNN
+F 1 "GND" H 7050 6850 50  0000 C CNN
+F 2 "" H 7050 7000 50  0000 C CNN
+F 3 "" H 7050 7000 50  0000 C CNN
+	1    7050 7000
+	1    0    0    -1
+$EndComp
+Wire Wire Line
+	7050 7000 7050 6950
+$Comp
+L Jumper_NO_Small JP1
+U 1 1 5A0F65B1
+P 6050 3850
+F 0 "JP1" H 6050 3930 50  0000 C CNN
+F 1 "Jumper_NO_Small" H 6060 3790 50  0001 C CNN
+F 2 "Resistors_SMD:R_0805_HandSoldering" H 6050 3850 50  0001 C CNN
+F 3 "" H 6050 3850 50  0000 C CNN
+	1    6050 3850
+	1    0    0    -1
+$EndComp
+Text HLabel 6150 3850 2    60   Input ~ 0
+MCU_VCC
 $EndSCHEMATC
