File: hardware/electronic/MK2/motor.sch (KiCad schematic (older format))
At the start: 7 parts, among them U1 TAMIYA_High_Speed_Gearbox, U3 Pololu_TB6612, U5 TB6612FNG

Commit message: HW: Update Mk-II design
Parts:
- removed C17, C18: 100nF, Capacitors_SMD:C_0805, symbol C_Small
- removed C19: 10uF 20V, Capacitors_Tantalum_SMD:TantalC_SizeT_EIA-3528, symbol CP1
- removed Encoder1: MOLEX 22-28-5044, Pin_Headers:Pin_Header_Straight_1x04, symbol CONN_01X04
- removed U1: TAMIYA_High_Speed_Gearbox, OPAVES_Footprints:TAMIYA_HIgh_Speed_Gearbox, symbol TAMIYA_High_Speed_Gearbox
- removed U5: TB6612FNG, Housings_SSOP:SSOP-24_5.3x8.2mm_Pitch0.65mm, symbol TB6612FNG
- added Motor_Left1, Motor_Right1: CONN_01X02, Pin_Headers:Pin_Header_Straight_1x02, symbol CONN_01X02
- renumbered U3 to U1
Connections:
- net MOTOR_A1: now also Motor_Left1.1 (P1)
- net MOTOR_A2: now also Motor_Left1.2 (P2)
- net MOTOR_B1: now also Motor_Right1.2 (P2)
- net MOTOR_B2: now also Motor_Right1.1 (P1)
Other:
- moved on the sheet: U1
