File: hardware/electronic/MK2/power.sch (KiCad schematic (older format))
At the start: 11 parts, among them U7 0S203013MT8QN1

Commit message: HW: Update Mk-II design
Parts:
- renumbered D4 to D1, D5 to D2, R3 to R1, R4 to R2, R15 to R3, R16 to R4, U7 to U2
Changed lines of the file:
@@
 Title "O'PAVES Mk-II"
 Date ""
-Rev "A"
+Rev "B"
 Comp "AdaCore"
 Comment1 "Licensed under CERN OHL v.1.2 or later"
@@
 $EndComp
 $Comp
-L GND #PWR07
+L GND #PWR03
 U 1 1 5885FB0A
 P 1650 2350
-F 0 "#PWR07" H 1650 2100 50  0001 C CNN
+F 0 "#PWR03" H 1650 2100 50  0001 C CNN
 F 1 "GND" H 1650 2200 50  0000 C CNN
 F 2 "" H 1650 2350 50  0000 C CNN
@@
 3 Cell NiMH:\n - Max: 4.5V\n - Typical: 3.6V\n - Low: 2.7V
 $Comp
-L R R3
+L R R1
 U 1 1 5885FCA2
 P 3300 2100
-F 0 "R3" V 3380 2100 50  0000 C CNN
+F 0 "R1" V 3380 2100 50  0000 C CNN
 F 1 "5k" V 3300 2100 50  0000 C CNN
 F 2 "Resistors_SMD:R_0805" V 3230 2100 50  0001 C CNN
@@
 $EndComp
 $Comp
-L R R4
+L R R2
 U 1 1 5885FCD9
 P 3300 2500
-F 0 "R4" V 3380 2500 50  0000 C CNN
+F 0 "R2" V 3380 2500 50  0000 C CNN
 F 1 "10k" V 3300 2500 50  0000 C CNN
 F 2 "Resistors_SMD:R_0805" V 3230 2500 50  0001 C CNN
@@
 Connection ~ 3300 2300
 $Comp
-L GND #PWR08
+L GND #PWR04
 U 1 1 5885FD97
 P 3300 2650
-F 0 "#PWR08" H 3300 2400 50  0001 C CNN
+F 0 "#PWR04" H 3300 2400 50  0001 C CNN
 F 1 "GND" H 3300 2500 50  0000 C CNN
 F 2 "" H 3300 2650 50  0000 C CNN
@@
 5V
 $Comp
-L GND #PWR09
+L GND #PWR05
 U 1 1 588A1F16
 P 7400 2800
-F 0 "#PWR09" H 7400 2550 50  0001 C CNN
+F 0 "#PWR05" H 7400 2550 50  0001 C CNN
 F 1 "GND" H 7400 2650 50  0000 C CNN
 F 2 "" H 7400 2800 50  0000 C CNN
@@
 3V3
 $Comp
-L GND #PWR010
+L GND #PWR06
 U 1 1 588A6FD6
 P 7150 6050
-F 0 "#PWR010" H 7150 5800 50  0001 C CNN
+F 0 "#PWR06" H 7150 5800 50  0001 C CNN
 F 1 "GND" H 7150 5900 50  0000 C CNN
 F 2 "" H 7150 6050 50  0000 C CNN
@@
 TODO: Reverse polarity protection (maybe)
 $Comp
-L Led_Small D4
+L Led_Small D1
 U 1 1 58DB4328
 P 6850 2350
-F 0 "D4" H 6800 2475 50  0000 L CNN
+F 0 "D1" H 6800 2475 50  0000 L CNN
 F 1 "Red" H 6800 2250 50  0000 L CNN
 F 2 "LEDs:LED_0805" V 6850 2350 50  0001 C CNN
@@
 $EndComp
 $Comp
-L R R15
+L R R3
 U 1 1 58DB4330
 P 6850 2600
-F 0 "R15" V 6930 2600 50  0000 C CNN
+F 0 "R3" V 6930 2600 50  0000 C CNN
 F 1 "330" V 6850 2600 50  0000 C CNN
 F 2 "Resistors_SMD:R_0805" V 6780 2600 50  0001 C CNN
@@
 Connection ~ 6850 2200
 $Comp
-L Led_Small D5
+L Led_Small D2
 U 1 1 58DB4F4F
 P 6850 5550
-F 0 "D5" H 6800 5675 50  0000 L CNN
+F 0 "D2" H 6800 5675 50  0000 L CNN
 F 1 "Green" H 6750 5450 50  0000 L CNN
 F 2 "LEDs:LED_0805" V 6850 5550 50  0001 C CNN
@@
 $EndComp
 $Comp
-L R R16
+L R R4
 U 1 1 58DB4F57
 P 6850 5800
-F 0 "R16" V 6930 5800 50  0000 C CNN
+F 0 "R4" V 6930 5800 50  0000 C CNN
 F 1 "330" V 6850 5800 50  0000 C CNN
 F 2 "Resistors_SMD:R_0805" V 6780 5800 50  0001 C CNN
@@
 Connection ~ 7150 5950
 $Comp
-L DP3T_switch U7
+L DP3T_switch U2
 U 1 1 58DB8591
 P 3000 4500
-F 0 "U7" H 3000 4500 60  0000 C CNN
+F 0 "U2" H 3000 4500 60  0000 C CNN
 F 1 "0S203013MT8QN1" H 3000 4400 60  0000 C CNN
 F 2 "OPAVES_Footprints:DP3T_switch" H 3000 4500 60  0001 C CNN
